File: pcb/CBI.kicad_pcb (KiCad board)
At the start: 2 copper layers, 43.8 x 31.8 mm, 87 parts, among them J1 Conn_01x03_Socket, J11 Screw_Terminal_01x03, J12 Conn_01x04_Pin, J4 Conn_01x02_Socket, J5 Conn_01x02_Socket, J6 Conn_01x03_Socket, J7 Conn_01x03_Socket, J9 Conn_01x02_Socket, J99 Conn_01x03_Socket, Q1 BC817, Q11 MMBFJ113, Q12 MMBFJ113, Q13 MMBFJ113, Q14 AO3416A, Q15 AO3416A, Q2 BC817, Q3 MMBFJ113, Q4 MMBFJ113, Q5 AO3416A, Q6 AO3416A, SW1 SW_SPST, U1 CNY17-4, U2 CNY17-4, U3 MCP23008-xSO

Commit message: Add missing vendor(id)
Parts:
- R5, R6: value 22 -> 22R
Changed lines of the file:
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@@
     (property "Sheetname" "")
     (property "Vendor" "HTL")
-    (property "VendorId" "102940")
+    (property "VendorId" "102919")
     (property "ki_description" "Resistor")
     (property "ki_keywords" "R res resistor")
@@
     (property "Sheetfile" "CBI.kicad_sch")
     (property "Sheetname" "")
+    (property "Vendor" "DigiKey")
+    (property "VendorId" "160-1323-5-ND")
     (property "ki_description" "DC Optocoupler Base Connected, Vce 70V, CTR 160-320%, Viso 5000V (RMS), DIP6")
     (property "ki_keywords" "NPN DC Optocoupler Base Connected")
@@
     (property "Sheetfile" "CBI.kicad_sch")
     (property "Sheetname" "")
+    (property "Vendor" "HTL")
+    (property "VendorId" "100187")
     (property "ki_description" "Zener diode")
     (property "ki_keywords" "diode")
@@
     (property "Sheetname" "")
     (property "Vendor" "HTL")
-    (property "VendorId" "102938")
+    (property "VendorId" "102951")
     (property "ki_description" "Resistor")
     (property "ki_keywords" "R res resistor")
@@
     (property "Sheetname" "")
     (property "Vendor" "HTL")
-    (property "VendorId" "102940")
+    (property "VendorId" "102919")
     (property "ki_description" "Resistor")
     (property "ki_keywords" "R res resistor")
@@
     (property "Sheetname" "")
     (property "Vendor" "HTL")
-    (property "VendorId" "102938")
+    (property "VendorId" "102951")
     (property "ki_description" "Resistor")
     (property "ki_keywords" "R res resistor")
@@
     (property "Sheetfile" "CBI.kicad_sch")
     (property "Sheetname" "")
+    (property "Vendor" "DigiKey")
+    (property "VendorId" "277-1151-ND, 277-1012-ND")
     (property "ki_description" "Generic screw terminal, single row, 01x03, script generated (kicad-library-utils/schlib/autogen/connector/)")
     (property "ki_keywords" "screw terminal")
@@
     (property "Sheetfile" "CBI.kicad_sch")
     (property "Sheetname" "")
+    (property "Vendor" "DigiKey")
+    (property "VendorId" "160-1323-5-ND")
     (property "ki_description" "DC Optocoupler Base Connected, Vce 70V, CTR 160-320%, Viso 5000V (RMS), DIP6")
     (property "ki_keywords" "NPN DC Optocoupler Base Connected")
@@
     (property "Sheetfile" "CBI.kicad_sch")
     (property "Sheetname" "")
+    (property "Vendor" "HTL")
+    (property "VendorId" "100187")
     (property "ki_description" "Zener diode")
     (property "ki_keywords" "diode")
@@
     (property "Sheetname" "")
     (property "Vendor" "HTL")
-    (property "VendorId" "102938")
+    (property "VendorId" "102951")
     (property "ki_description" "Resistor")
     (property "ki_keywords" "R res resistor")
@@
     (property "Sheetname" "")
     (property "Vendor" "HTL")
-    (property "VendorId" "102938")
+    (property "VendorId" "102951")
     (property "ki_description" "Resistor")
     (property "ki_keywords" "R res resistor")
@@
     (property "Sheetname" "")
     (property "Vendor" "HTL")
-    (property "VendorId" "102938")
+    (property "VendorId" "102937")
     (property "ki_description" "Resistor")
     (property "ki_keywords" "R res resistor")
@@
     (property "Sheetname" "")
     (property "Vendor" "HTL")
-    (property "VendorId" "102938")
+    (property "VendorId" "102919")
     (property "ki_description" "Resistor")
     (property "ki_keywords" "R res resistor")
@@
         (effects (font (size 0.6 0.6) (thickness 0.12)) (justify mirror))
     )
-    (fp_text value "22" (at 0 1.6256) (layer "B.Fab")
+    (fp_text value "22R" (at 0 1.6256) (layer "B.Fab")
         (effects (font (size 1 1) (thickness 0.15)) (justify mirror))
     )
@@
     (property "Sheetname" "")
     (property "Vendor" "HTL")
-    (property "VendorId" "102938")
+    (property "VendorId" "102951")
     (property "ki_description" "Resistor")
     (property "ki_keywords" "R res resistor")
@@
     (property "Sheetfile" "CBI.kicad_sch")
     (property "Sheetname" "")
+    (property "Vendor" "HTL")
+    (property "VendorId" "103452")
     (property "ki_description" "0.8A Ic, 45V Vce, NPN Transistor, SOT-23")
     (property "ki_keywords" "NPN Transistor")
@@
     (property "Sheetname" "")
     (property "Vendor" "HTL")
-    (property "VendorId" "102938")
+    (property "VendorId" "102937")
     (property "ki_description" "Resistor")
     (property "ki_keywords" "R res resistor")
@@
     (property "Sheetfile" "CBI.kicad_sch")
     (property "Sheetname" "")
+    (property "Vendor" "HTL")
+    (property "VendorId" "103452")
     (property "ki_description" "0.8A Ic, 45V Vce, NPN Transistor, SOT-23")
     (property "ki_keywords" "NPN Transistor")
@@
     (property "Sheetname" "")
     (property "Vendor" "HTL")
-    (property "VendorId" "102940")
+    (property "VendorId" "102951")
     (property "ki_description" "Resistor")
     (property "ki_keywords" "R res resistor")
@@
     (property "Sheetfile" "CBI.kicad_sch")
     (property "Sheetname" "")
+    (property "Vendor" "HTL")
+    (property "VendorId" "100187")
     (property "ki_description" "Zener diode")
     (property "ki_keywords" "diode")
@@
     (property "Sheetname" "")
     (property "Vendor" "HTL")
-    (property "VendorId" "102938")
+    (property "VendorId" "102951")
     (property "ki_description" "Resistor")
     (property "ki_keywords" "R res resistor")
@@
     (property "Sheetname" "")
     (property "Vendor" "HTL")
-    (property "VendorId" "102940")
+    (property "VendorId" "102951")
     (property "ki_description" "Resistor")
     (property "ki_keywords" "R res resistor")
@@
     (property "Sheetfile" "CBI.kicad_sch")
     (property "Sheetname" "")
+    (property "Vendor" "HTL")
+    (property "VendorId" "100187")
     (property "ki_description" "Zener diode")
     (property "ki_keywords" "diode")
@@
     (property "Sheetname" "")
     (property "Vendor" "HTL")
-    (property "VendorId" "102938")
+    (property "VendorId" "102919")
     (property "ki_description" "Resistor")
     (property "ki_keywords" "R res resistor")
@@
         (effects (font (size 0.6 0.6) (thickness 0.12)) (justify mirror))
     )
-    (fp_text value "22" (at 0 -1.5748) (layer "B.Fab")
+    (fp_text value "22R" (at 0 -1.5748) (layer "B.Fab")
         (effects (font (size 1 1) (thickness 0.15)) (justify mirror))
     )
