File: pcb/CBI.kicad_sch (KiCad schematic)
At the start: 87 parts, among them J1 Conn_01x03_Socket, J11 Screw_Terminal_01x03, J12 Conn_01x04_Pin, J4 Conn_01x02_Socket, J5 Conn_01x02_Socket, J6 Conn_01x03_Socket, J7 Conn_01x03_Socket, J9 Conn_01x02_Socket, J99 Conn_01x03_Socket, Q1 BC817, Q11 MMBFJ113, Q12 MMBFJ113, Q13 MMBFJ113, Q14 AO3416A, Q15 AO3416A, Q2 BC817, Q3 MMBFJ113, Q4 MMBFJ113, Q5 AO3416A, Q6 AO3416A, SW1 SW_SPST, U1 CNY17-4, U2 CNY17-4, U3 MCP23008-xSO

Commit message: Update to KiCAD 9
Parts:
- FID1, FID2, FID3, FID4: now left out of the parts list

Commit message: Rename/Add/Remove bom fields
Parts:
- C1: HTL (none) -> 103620; Vendor HTL -> (none); VendorId 103620 -> (none)
- C2, C3, C5, C6: HTL (none) -> 100128; Vendor HTL -> (none); VendorId 100128 -> (none)
- D1, D10, D11, D12, D13, D14, D2, D5, D6, D7, D8, D9: HTL (none) -> 100206; Vendor HTL -> (none); VendorId 100206 -> (none)
- D15: HTL (none) -> 100457; Vendor HTL -> (none); VendorId 100457 -> (none)
- D16, D17: HTL (none) -> 100459; Vendor HTL -> (none); VendorId 100459 -> (none)
- D18, D19, D3, D4: HTL (none) -> 100458; Vendor HTL -> (none); VendorId 100458 -> (none)
- D20, D21, D22, D23: HTL (none) -> 100187; Vendor HTL -> (none); VendorId 100187 -> (none)
- J1, J6, J7, J99: DigiKey (none) -> 2057-RS1-03-G-ND; Vendor DigiKey -> (none); VendorId 2057-RS1-03-G-ND -> (none)
- J11: DigiKey (none) -> 277-1151-ND, 277-1012-ND; Vendor DigiKey -> (none); VendorId 277-1151-ND, 277-1012-ND -> (none)
- J12: HTL (none) -> 101521; Vendor HTL -> (none); VendorId 101521 -> (none)
- J4, J5, J9: DigiKey (none) -> 2057-RS1-02-G-ND; Vendor DigiKey -> (none); VendorId 2057-RS1-02-G-ND -> (none)
- Q1, Q2: HTL (none) -> 103452; Vendor HTL -> (none); VendorId 103452 -> (none)
- Q11, Q12, Q13, Q3, Q4: DigiKey (none) -> MMBFJ113CT-ND; Vendor DigiKey -> (none); VendorId MMBFJ113CT-ND -> (none)
- Q14, Q15, Q5, Q6: HTL (none) -> 103512; Vendor HTL -> (none); VendorId 103512 -> (none)
- R1, R10, R22, R24, R26, R28, R3, R9: HTL (none) -> 102951; Vendor HTL -> (none); VendorId 102951 -> (none)
- R11, R12, R5, R6: HTL (none) -> 102919; Vendor HTL -> (none); VendorId 102919 -> (none)
- R13, R14, R34, R35: HTL (none) -> 102940; Vendor HTL -> (none); VendorId 102940 -> (none)
- R15, R16, R21, R31, R7, R8: HTL (none) -> 102961; Vendor HTL -> (none); VendorId 102961 -> (none)
- R2, R4: HTL (none) -> 102937; Vendor HTL -> (none); VendorId 102937 -> (none)
- R30: HTL (none) -> 102973; Vendor HTL -> (none); VendorId 102973 -> (none)
- R32: HTL (none) -> 102956; Vendor HTL -> (none); VendorId 102956 -> (none)
- R33: HTL (none) -> 102959; Vendor HTL -> (none); VendorId 102959 -> (none)
- R36, R37, R38: HTL (none) -> 102938; Vendor HTL -> (none); VendorId 102938 -> (none)
- SW1: HTL (none) -> 101614; Vendor HTL -> (none); VendorId 101614 -> (none)
- U1, U2: DigiKey (none) -> 160-1323-5-ND; Vendor DigiKey -> (none); VendorId 160-1323-5-ND -> (none)
- U3: DigiKey (none) -> MCP23008-E/SO-ND; Vendor DigiKey -> (none); VendorId MCP23008-E/SO-ND -> (none)
